File: circuit/thermometer.kicad_sch (KiCad schematic)
At the start: 35 parts, among them IC1 ICL7107CPL, IC2 TMP36, IC3 LM285Z-1.2, IC4 4001, SW1 SW_DIP_x04

Commit message: Finish off the PCB
Parts:
- removed SW1: SW_DIP_x04, Button_Switch_THT:SW_DIP_SPSTx04_Slide_9.78x12.34mm_W7.62mm_P2.54mm, symbol Switch:SW_DIP_x04
- added C10, C11: 47nF, Capacitor_THT:C_Disc_D4.3mm_W1.9mm_P5.00mm, symbol Device:C
- added J3: +5V, Connector_Wire:SolderWire-0.5sqmm_1x01_D0.9mm_OD2.1mm, symbol Connector_Generic:Conn_01x01
- added J4: GND, Connector_Wire:SolderWire-0.5sqmm_1x01_D0.9mm_OD2.1mm, symbol Connector_Generic:Conn_01x01
- added J5: ~, Connector_PinHeader_2.54mm:PinHeader_2x04_P2.54mm_Vertical, symbol Connector_Generic:Conn_02x04_Odd_Even
- C4: value 470nF -> 47nF
- C6: footprint Capacitor_THT:CP_Radial_Tantal_D4.5mm_P2.50mm -> Capacitor_THT:CP_Radial_D5.0mm_P2.50mm
- IC2: renamed from IC4; footprint Package_DIP:DIP-14_W7.62mm_Socket_LongPads -> Package_DIP:DIP-14_W7.62mm_LongPads
- IC2: renamed from IC4; footprint (none) -> Package_DIP:DIP-14_W7.62mm_LongPads
- renumbered IC2 to IC4
Connections:
- net +5V: now also DISP1.13 (ca2), DISP1.14 (ca1), C10.1, C11.1, J3.1 (Pin_1)
- net GND: now also C10.2, C11.2, J4.1 (Pin_1), J5.1 (Pin_1), J5.3 (Pin_3), J5.5 (Pin_5), J5.7 (Pin_7)
- net at R12.2: now also J5.6 (Pin_6)
- net at R13.2: now also J5.8 (Pin_8)
- net at R11.2: now also J5.4 (Pin_4)
- net at R10.1: now also J5.2 (Pin_2)
- net at DISP1.5 (e2): now also IC1.18 (E3)
- net at IC1.2 (D1): now also DISP2.6 (d2)
Other:
- moved on the sheet: C3, IC2D

Commit message: A bit more tidying up
Parts:
- removed C3: 1uF, Capacitor_THT:C_Disc_D4.3mm_W1.9mm_P5.00mm, symbol Device:C_Small
- added C5: 10nF, Capacitor_THT:C_Disc_D4.3mm_W1.9mm_P5.00mm, symbol Device:C_Small
- renumbered C8 to C10, C9 to C11, C4 to C3, C5 to C4, C7 to C6, C6 to C7, C11 to C8, C10 to C9, J5 to J2, J2 to J5, R5 to R10, R6 to R11, R7 to R12, R8 to R13, R10 to R3, R11 to R4, R12 to R5, R13 to R6, R3 to R7, R4 to R8
Connections:
- net at IC1.31 (IN_HI), J1.2 (Pin_2): now also C5.2
- net at IC1.30 (IN_LO), J1.1 (Pin_1): now also C5.1
Other:
- moved on the sheet: C9, IC2C, IC2D
